File: eagle/current.brd (EAGLE design)
At the start: 50.5 x 50.8 mm, 39 parts, among them J2 3-pol, J3 3-pol, J4 3-pol, U2 ATMEGA328P_TQFP, Y1 16MHz

Commit message: Board upgrades
Parts:
- removed H3: MOUNT-PAD-ROUND3.6, holes:3,6-PAD
- added C10, C7, C8, C9: 10uF, SparkFun-Capacitors:EIA3216
- added IC1: REG1117, burr-brown:SOT223
- added SV3: (no value), con-lstb:MA04-2
- moved H2 43.7 mm to (5.84, 38.9)
- moved H4 1.63 mm to (6.10, 6.10)
- moved D1 1.52 mm to (28.7, 47.2)
- moved R14 1.44 mm to (32.8, 46.3)
- moved R15 1.43 mm to (32.8, 48.3)
- moved X1 1.02 mm to (22.5, 5.79)
- moved R13 0.83 mm to (24.8, 47.1)
- moved H1 0.36 mm to (45.0, 45.7)
- moved C4 0.15 mm to (24.5, 37.8)
Connections:
- new net 3V3: C10.+, IC1.2, SV3.1
- net A01: now also SV3.8
- net D00: now also SV3.7
- net D01: now also SV3.6
- net D02: now also SV3.5
- net GND: now also C10.-, C7.-, C8.-, C9.-, IC1.1, SV3.2, SV3.4
- net VCC: now also C7.+, C8.+, C9.+, IC1.3, SV3.3
Routing:
- net VCC: track 110.9 -> 161.8 mm, vias 3 -> 5
- net RESET: track 0.00 -> 28.0 mm, vias 0 -> 1
- net D02: track 0.00 -> 21.2 mm, vias 0 -> 1
- net D00: track 0.00 -> 18.8 mm, vias 0 -> 1
- net D01: track 0.00 -> 17.1 mm, vias 0 -> 1
- net 3V3: track 0.00 -> 11.6 mm
- net D07: track 21.7 -> 32.1 mm, vias 1 -> 2
- net A01: track 0.00 -> 7.70 mm
- net D05: track 19.6 -> 20.9 mm
- net D06: track 23.0 -> 24.2 mm
- net D08: track 34.5 -> 33.8 mm
- net N$4: track 1.76 -> 2.40 mm
