File: eagle/current.sch (EAGLE design)
At the start: 39 parts, among them J2 3-pol, J3 3-pol, J4 3-pol, U2 ATMEGA328P_TQFP, Y1 16MHz

Commit message: Board upgrades
Parts:
- removed H3: MOUNT-PAD-ROUND3.6, holes:MOUNT-PAD-ROUND3.6
- added C10, C7, C8, C9: 10uF, SparkFun-Capacitors:10UF-POLAR-EIA3216-16V-10%(TANT)
- added IC1: REG1117, burr-brown:REG1117
- added SV3: (no value), con-lstb:MA04-2
Connections:
- new net 3V3: C10.+, IC1.VOUT, SV3.1
- net A01: now also SV3.8
- net D00: now also SV3.7
- net D01: now also SV3.6
- net D02: now also SV3.5
- net GND: now also C10.-, C7.-, C8.-, C9.-, IC1.GND, SV3.2, SV3.4
- net VCC: now also C7.+, C8.+, C9.+, IC1.VIN, SV3.3
Changed lines of the file:
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@@
 <part name="Y1" library="SparkFun-Clocks" deviceset="CRYSTAL" device="SMD-3.2X2.5" value="16MHz"/>
 <part name="H2" library="holes" deviceset="MOUNT-PAD-ROUND" device="3.6"/>
-<part name="H3" library="holes" deviceset="MOUNT-PAD-ROUND" device="3.6"/>
 <part name="H4" library="holes" deviceset="MOUNT-PAD-ROUND" device="3.6"/>
 <part name="X1" library="con-wago-500" library_urn="urn:adsk.eagle:library:195" deviceset="W237-102" device="" package3d_urn="urn:adsk.eagle:package:10688/1"/>
+<part name="SV3" library="con-lstb" library_urn="urn:adsk.eagle:library:162" deviceset="MA04-2" device="" package3d_urn="urn:adsk.eagle:package:8368/1"/>
+<part name="C7" library="SparkFun-Capacitors" deviceset="10UF-POLAR" device="-EIA3216-16V-10%(TANT)" value="10uF"/>
+<part name="C8" library="SparkFun-Capacitors" deviceset="10UF-POLAR" device="-EIA3216-16V-10%(TANT)" value="10uF"/>
+<part name="IC1" library="burr-brown" library_urn="urn:adsk.eagle:library:111" deviceset="REG1117" device="" package3d_urn="urn:adsk.eagle:package:4940/1"/>
+<part name="C9" library="SparkFun-Capacitors" deviceset="10UF-POLAR" device="-EIA3216-16V-10%(TANT)" value="10uF"/>
+<part name="C10" library="SparkFun-Capacitors" deviceset="10UF-POLAR" device="-EIA3216-16V-10%(TANT)" value="10uF"/>
 </parts>
 <sheets>
@@
 <attribute name="VALUE" x="73.914" y="81.3562" size="1.778" layer="96"/>
 </instance>
-<instance part="H3" gate="G$1" x="91.44" y="81.28" smashed="yes">
-<attribute name="NAME" x="94.234" y="81.8642" size="1.778" layer="95"/>
-<attribute name="VALUE" x="94.234" y="78.8162" size="1.778" layer="96"/>
-</instance>
 <instance part="H4" gate="G$1" x="109.22" y="93.98" smashed="yes">
 <attribute name="NAME" x="112.014" y="94.5642" size="1.778" layer="95"/>
@@
 <attribute name="VALUE" x="152.4" y="115.443" size="1.778" layer="96" rot="R180"/>
 <attribute name="NAME" x="149.86" y="110.871" size="1.778" layer="95"/>
+</instance>
+<instance part="SV3" gate="G$1" x="111.76" y="33.02" smashed="yes">
+<attribute name="VALUE" x="107.95" y="25.4" size="1.778" layer="96"/>
+<attribute name="NAME" x="107.95" y="38.862" size="1.778" layer="95"/>
+</instance>
+<instance part="C7" gate="G$1" x="7.62" y="40.64" smashed="yes">
+<attribute name="NAME" x="8.636" y="41.275" size="1.778" layer="95"/>
+<attribute name="VALUE" x="8.636" y="36.449" size="1.778" layer="96"/>
+</instance>
+<instance part="C8" gate="G$1" x="0" y="40.64" smashed="yes">
+<attribute name="NAME" x="1.016" y="41.275" size="1.778" layer="95"/>
+<attribute name="VALUE" x="1.016" y="36.449" size="1.778" layer="96"/>
+</instance>
+<instance part="IC1" gate="G$1" x="210.82" y="71.12" smashed="yes">
+<attribute name="NAME" x="203.2" y="76.835" size="1.778" layer="95" ratio="10"/>
+<attribute name="VALUE" x="205.74" y="73.66" size="1.778" layer="96" ratio="10"/>
+</instance>
+<instance part="C9" gate="G$1" x="195.58" y="68.58" smashed="yes">
+<attribute name="NAME" x="196.596" y="69.215" size="1.778" layer="95"/>
+<attribute name="VALUE" x="196.596" y="64.389" size="1.778" layer="96"/>
+</instance>
+<instance part="C10" gate="G$1" x="226.06" y="68.58" smashed="yes">
+<attribute name="NAME" x="227.076" y="69.215" size="1.778" layer="95"/>
+<attribute name="VALUE" x="227.076" y="64.389" size="1.778" layer="96"/>
 </instance>
 </instances>
@@
 </segment>
 <segment>
+<pinref part="U2" gate="U1" pin="GND"/>
+<wire x1="45.72" y1="2.54" x2="40.64" y2="2.54" width="0.1524" layer="91"/>
+<label x="38.1" y="2.54" size="1.778" layer="95"/>
+</segment>
+<segment>
+<pinref part="X1" gate="-2" pin="KL"/>
+<wire x1="144.78" y1="111.76" x2="137.16" y2="111.76" width="0.1524" layer="91"/>
+<label x="139.7" y="111.76" size="1.778" layer="95"/>
+</segment>
+<segment>
+<pinref part="C8" gate="G$1" pin="-"/>
+<wire x1="0" y1="35.56" x2="0" y2="22.86" width="0.1524" layer="91"/>
+<pinref part="C7" gate="G$1" pin="-"/>
+<wire x1="7.62" y1="35.56" x2="7.62" y2="22.86" width="0.1524" layer="91"/>
+<wire x1="0" y1="22.86" x2="7.62" y2="22.86" width="0.1524" layer="91"/>
 <pinref part="U2" gate="U1" pin="AGND"/>
 <label x="40.64" y="5.08" size="1.778" layer="95"/>
@@
 <wire x1="27.94" y1="5.08" x2="27.94" y2="22.86" width="0.1524" layer="91"/>
 <junction x="27.94" y="22.86"/>
-</segment>
-<segment>
-<pinref part="U2" gate="U1" pin="GND"/>
-<wire x1="45.72" y1="2.54" x2="40.64" y2="2.54" width="0.1524" layer="91"/>
-<label x="38.1" y="2.54" size="1.778" layer="95"/>
-</segment>
-<segment>
-<pinref part="X1" gate="-2" pin="KL"/>
-<wire x1="144.78" y1="111.76" x2="137.16" y2="111.76" width="0.1524" layer="91"/>
-<label x="139.7" y="111.76" size="1.778" layer="95"/>
+<wire x1="7.62" y1="22.86" x2="15.24" y2="22.86" width="0.1524" layer="91"/>
+<junction x="7.62" y="22.86"/>
+<junction x="15.24" y="22.86"/>
+</segment>
+<segment>
+<pinref part="IC1" gate="G$1" pin="GND"/>
+<wire x1="210.82" y1="58.42" x2="210.82" y2="55.88" width="0.1524" layer="91"/>
+<label x="210.82" y="55.88" size="1.778" layer="95"/>
+<pinref part="C9" gate="G$1" pin="-"/>
+<wire x1="195.58" y1="63.5" x2="195.58" y2="55.88" width="0.1524" layer="91"/>
+<wire x1="195.58" y1="55.88" x2="210.82" y2="55.88" width="0.1524" layer="91"/>
+<pinref part="C10" gate="G$1" pin="-"/>
+<wire x1="210.82" y1="55.88" x2="226.06" y2="55.88" width="0.1524" layer="91"/>
+<wire x1="226.06" y1="55.88" x2="226.06" y2="63.5" width="0.1524" layer="91"/>
+<junction x="210.82" y="55.88"/>
+</segment>
+<segment>
+<pinref part="SV3" gate="G$1" pin="4"/>
+<wire x1="104.14" y1="30.48" x2="101.6" y2="30.48" width="0.1524" layer="91"/>
+<label x="101.6" y="30.48" size="1.778" layer="95"/>
+</segment>
+<segment>
+<pinref part="SV3" gate="G$1" pin="2"/>
+<wire x1="104.14" y1="27.94" x2="101.6" y2="27.94" width="0.1524" layer="91"/>
+<label x="101.6" y="27.94" size="1.778" layer="95"/>
 </segment>
 </net>
@@
 <wire x1="33.02" y1="53.34" x2="33.02" y2="55.88" width="0.1524" layer="91"/>
 <junction x="33.02" y="55.88"/>
+<pinref part="C7" gate="G$1" pin="+"/>
+<wire x1="7.62" y1="60.96" x2="7.62" y2="43.18" width="0.1524" layer="91"/>
+<wire x1="15.24" y1="60.96" x2="7.62" y2="60.96" width="0.1524" layer="91"/>
+<pinref part="C8" gate="G$1" pin="+"/>
+<wire x1="0" y1="60.96" x2="0" y2="43.18" width="0.1524" layer="91"/>
+<wire x1="0" y1="60.96" x2="7.62" y2="60.96" width="0.1524" layer="91"/>
+<junction x="7.62" y="60.96"/>
 </segment>
 <segment>
@@
 <label x="154.94" y="144.78" size="1.778" layer="95"/>
 </segment>
+<segment>
+<pinref part="IC1" gate="G$1" pin="VIN"/>
+<wire x1="198.12" y1="71.12" x2="195.58" y2="71.12" width="0.1524" layer="91"/>
+<label x="193.04" y="71.12" size="1.778" layer="95"/>
+<pinref part="C9" gate="G$1" pin="+"/>
+<wire x1="195.58" y1="71.12" x2="193.04" y2="71.12" width="0.1524" layer="91"/>
+<junction x="195.58" y="71.12"/>
+</segment>
+<segment>
+<pinref part="SV3" gate="G$1" pin="3"/>
+<wire x1="119.38" y1="30.48" x2="121.92" y2="30.48" width="0.1524" layer="91"/>
+<label x="119.38" y="30.48" size="1.778" layer="95"/>
+</segment>
 </net>
 <net name="RESET" class="0">
@@
 <wire x1="88.9" y1="58.42" x2="93.98" y2="58.42" width="0.1524" layer="91"/>
 <label x="91.44" y="58.42" size="1.778" layer="95"/>
+</segment>
+<segment>
+<pinref part="SV3" gate="G$1" pin="8"/>
+<wire x1="104.14" y1="35.56" x2="101.6" y2="35.56" width="0.1524" layer="91"/>
+<label x="101.6" y="35.56" size="1.778" layer="95"/>
 </segment>
 </net>
@@
 <label x="91.44" y="38.1" size="1.778" layer="95"/>
 </segment>
+<segment>
+<pinref part="SV3" gate="G$1" pin="7"/>
+<wire x1="119.38" y1="35.56" x2="121.92" y2="35.56" width="0.1524" layer="91"/>
+<label x="119.38" y="35.56" size="1.778" layer="95"/>
+</segment>
 </net>
 <net name="D01" class="0">
@@
 <label x="91.44" y="35.56" size="1.778" layer="95"/>
 </segment>
+<segment>
+<pinref part="SV3" gate="G$1" pin="6"/>
+<wire x1="104.14" y1="33.02" x2="101.6" y2="33.02" width="0.1524" layer="91"/>
+<label x="101.6" y="33.02" size="1.778" layer="95"/>
+</segment>
 </net>
 <net name="D02" class="0">
@@
 <wire x1="88.9" y1="33.02" x2="93.98" y2="33.02" width="0.1524" layer="91"/>
 <label x="91.44" y="33.02" size="1.778" layer="95"/>
+</segment>
+<segment>
+<pinref part="SV3" gate="G$1" pin="5"/>
+<wire x1="119.38" y1="33.02" x2="121.92" y2="33.02" width="0.1524" layer="91"/>
+<label x="119.38" y="33.02" size="1.778" layer="95"/>
 </segment>
 </net>
@@
 </segment>
 </net>
+<net name="3V3" class="0">
+<segment>
+<pinref part="IC1" gate="G$1" pin="VOUT"/>
+<wire x1="223.52" y1="71.12" x2="226.06" y2="71.12" width="0.1524" layer="91"/>
+<label x="226.06" y="71.12" size="1.778" layer="95"/>
+<pinref part="C10" gate="G$1" pin="+"/>
+<wire x1="226.06" y1="71.12" x2="228.6" y2="71.12" width="0.1524" layer="91"/>
+<junction x="226.06" y="71.12"/>
+</segment>
+<segment>
+<pinref part="SV3" gate="G$1" pin="1"/>
+<wire x1="119.38" y1="27.94" x2="121.92" y2="27.94" width="0.1524" layer="91"/>
+<label x="119.38" y="27.94" size="1.778" layer="95"/>
+</segment>
+</net>
